File: hardware/OricMouse.kicad_pcb (KiCad board)
At the start: 2 copper layers, 85.1 x 71.1 mm, 43 parts, among them P1 CONN_02X17, P2 PROP PLUG, P3 PS2/0, P4 PS2 / 1, P5 ADB, P6 EXPANSION, Q1 BS170, Q2 BS170, Q3 BS170, Q4 BS170, Q5 BS170, Q6 BS170, SW1 RESET, U1 P8X32A, U2 24C512, U3 LD1117, U4 74LVC245, U5 74LVC244, U6 74LVC244, Y1 5MHz

Commit message: Add latest changes from 08/11/2015
Parts:
- moved C3 0.64 mm to (156.8, 122.0)
- renumbered REF** to Hole1, REF** to Hole2, REF** to Hole3, REF** to Hole4, REF** to OSHW
Routing:
- net /~RST: track 131.5 -> 136.5 mm
- net +3V3: track 119.4 -> 117.5 mm
- net /~RESET: track 40.2 -> 39.2 mm
- net /mRW: track 48.0 -> 48.9 mm, vias 1 -> 0
- net /mIOc: track 39.0 -> 39.4 mm, vias 1 -> 0
Other:
- board text added: "OricMouse Rev 1.0 08/11/2015"
- board text removed: "OricMouse Rev 1.0 01/11/2015"
