File: hardware/OricMouse.sch (KiCad schematic (older format))
At the start: 37 parts, among them P1 CONN_02X17, P2 PROP PLUG, P3 PS2 / 0, P4 PS2 / 1, P5 ADB, P6 EXP, Q1 BS170, Q2 BS170, Q3 BS170, Q4 BS170, Q5 BS170, Q6 BS170, SW1 RESET, U1 P8X32A, U2 24C512, U3 LM2931AZ-3.3/5.0, U4 74LVC245, U5 74LVC244, U6 74LVC244, Y1 5MHz

Commit message: Add latest changes from 08/11/2015
Parts:
- added R14: 10K, Resistors_ThroughHole:Resistor_Vertical_RM5mm, symbol R
Connections:
- net +3V3: now also R14.1
- net SCL: now also R14.2
Changed lines of the file:
@@
 	7000 3900 7000 3950
 Wire Wire Line
-	7000 5550 7250 5550
+	7000 5550 7500 5550
 Wire Wire Line
 	1250 3350 1250 3200
@@
 Text Label 8150 5050 0    60   ~ 0
 mPhi2
+$Comp
+L R R14
+U 1 1 564125B0
+P 7700 5400
+F 0 "R14" V 7600 5400 50  0000 C CNN
+F 1 "10K" V 7700 5400 50  0000 C CNN
+F 2 "Resistors_ThroughHole:Resistor_Vertical_RM5mm" V 7630 5400 30  0001 C CNN
+F 3 "" H 7700 5400 30  0000 C CNN
+	1    7700 5400
+	0    1    1    0
+$EndComp
+Wire Wire Line
+	7500 5550 7500 5400
+Wire Wire Line
+	7500 5400 7550 5400
+Wire Wire Line
+	7850 5400 8050 5400
+Wire Wire Line
+	8050 5400 8050 5300
+Connection ~ 8050 5300
 $EndSCHEMATC
